File: din13f-breakout.kicad_pcb (KiCad board)
At the start: 2 copper layers, 37.8 x 42.7 mm, 5 parts, among them J1 DB15_Female_HighDensity, J2 RCJ-017, J3 Conn_01x13, J4 SDD-130J

Commit message: v0.1 board
Routing:
- net /AUDIO_IN: vias 3 -> 2
Changed lines of the file:
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@@
       (outputformat 1)
       (mirror false)
-      (drillshape 1)
+      (drillshape 0)
       (scaleselection 1)
-      (outputdirectory "")
+      (outputdirectory "st-13f-breakout-v0.1")
     )
   )
@@
       (effects (font (size 1 1) (thickness 0.15)))
     )
-    (fp_text user "*" (at 0 0) (layer "F.SilkS")
+    (fp_text user "*" (at 0 0) (layer "F.SilkS") hide
       (effects (font (size 1 1) (thickness 0.15)))
     )
@@
   (segment (start 145.868 101.062) (end 145.868 100.562) (width 1.5) (layer "B.Cu") (net 6))
   (segment (start 145.868 100.562) (end 150.368 96.062) (width 1.5) (layer "B.Cu") (net 6))
-  (segment (start 137.16 87.549228) (end 137.16 88.9) (width 0.25) (layer "F.Cu") (net 9))
+  (segment (start 137.16 87.549228) (end 137.16 90.17) (width 0.25) (layer "F.Cu") (net 9))
   (segment (start 135.881872 86.2711) (end 137.16 87.549228) (width 0.25) (layer "F.Cu") (net 9))
-  (segment (start 137.16 88.9) (end 137.16 90.17) (width 0.25) (layer "F.Cu") (net 9))
   (segment (start 137.16 90.17) (end 135.636 91.694) (width 0.25) (layer "F.Cu") (net 9))
   (segment (start 135.636 91.694) (end 135.636 97.536) (width 0.25) (layer "F.Cu") (net 9))
@@
   (segment (start 121.666 91.44) (end 121.666 87.376) (width 0.25) (layer "F.Cu") (net 16))
   (via (at 121.666 91.44) (size 0.8) (drill 0.4) (layers "F.Cu" "B.Cu") (net 16))
-  (via (at 119.38 85.09) (size 0.8) (drill 0.4) (layers "F.Cu" "B.Cu") (net 16))
   (via (at 135.89 88.646) (size 0.8) (drill 0.4) (layers "F.Cu" "B.Cu") (net 16))
   (segment (start 131.064 88.646) (end 128.27 91.44) (width 0.25) (layer "B.Cu") (net 16))
