File: din13f-breakout.kicad_sch (KiCad schematic)
At the start: 5 parts

Commit message: v0.1 board
Parts:
- gave numbers to parts that had none: 5
Changed lines of the file:
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@@
   (symbol (lib_id "SDD-130J:SDD-130J") (at 184.15 72.39 0) (unit 1)
     (in_bom yes) (on_board yes) (fields_autoplaced)
-    (property "Reference" "J?" (id 0) (at 190.5 71.1199 0)
+    (property "Reference" "J4" (id 0) (at 190.5 71.1199 0)
       (effects (font (size 1.27 1.27)) (justify left))
     )
@@
   (symbol (lib_id "Connector:TestPoint") (at 167.005 95.885 180) (unit 1)
     (in_bom yes) (on_board yes) (fields_autoplaced)
-    (property "Reference" "TP?" (id 0) (at 168.91 97.9169 0)
+    (property "Reference" "TP1" (id 0) (at 168.91 97.9169 0)
       (effects (font (size 1.27 1.27)) (justify right))
     )
@@
   (symbol (lib_id "Connector:DB15_Female_HighDensity") (at 93.345 85.09 0) (unit 1)
     (in_bom yes) (on_board yes) (fields_autoplaced)
-    (property "Reference" "J?" (id 0) (at 93.345 62.23 0))
+    (property "Reference" "J1" (id 0) (at 93.345 62.23 0))
     (property "Value" "DB15_Female_HighDensity" (id 1) (at 93.345 64.77 0))
     (property "Footprint" "Connector_TE_AMP_HD15:FIXED-1-1734530-1" (id 2) (at 69.215 74.93 0)
@@
   (symbol (lib_id "RCJ-017:RCJ-017") (at 114.3 43.815 180) (unit 1)
     (in_bom yes) (on_board yes) (fields_autoplaced)
-    (property "Reference" "J?" (id 0) (at 119.38 42.5449 0)
+    (property "Reference" "J2" (id 0) (at 119.38 42.5449 0)
       (effects (font (size 1.27 1.27)) (justify right))
     )
@@
   (symbol (lib_id "Connector_Generic:Conn_01x13") (at 146.05 69.85 0) (mirror y) (unit 1)
     (in_bom yes) (on_board yes) (fields_autoplaced)
-    (property "Reference" "J?" (id 0) (at 146.05 48.26 0))
+    (property "Reference" "J3" (id 0) (at 146.05 48.26 0))
     (property "Value" "Conn_01x13" (id 1) (at 146.05 50.8 0))
     (property "Footprint" "Connectors:13p_GrabPads" (id 2) (at 146.05 69.85 0)
@@
   )
   (symbol_instances
-    (path "/29734604-6efb-4639-86ae-3538635da170"
-      (reference "J?") (unit 1) (value "SDD-130J") (footprint "CUI_SDD-130J")
-    )
     (path "/71981395-6e2d-465a-92b8-5b6eaab7b637"
-      (reference "J?") (unit 1) (value "DB15_Female_HighDensity") (footprint "Connector_TE_AMP_HD15:FIXED-1-1734530-1")
+      (reference "J1") (unit 1) (value "DB15_Female_HighDensity") (footprint "Connector_TE_AMP_HD15:FIXED-1-1734530-1")
     )
     (path "/eb7b1130-a3c5-419d-b014-6cc61228ef22"
-      (reference "J?") (unit 1) (value "RCJ-017") (footprint "Jacks:CUI_RCJ-017")
+      (reference "J2") (unit 1) (value "RCJ-017") (footprint "Jacks:CUI_RCJ-017")
     )
     (path "/eeb10296-3e7b-45d5-baab-9125e0c38015"
-      (reference "J?") (unit 1) (value "Conn_01x13") (footprint "Connectors:13p_GrabPads")
+      (reference "J3") (unit 1) (value "Conn_01x13") (footprint "Connectors:13p_GrabPads")
+    )
+    (path "/29734604-6efb-4639-86ae-3538635da170"
+      (reference "J4") (unit 1) (value "SDD-130J") (footprint "CUI_SDD-130J")
     )
     (path "/3a31be16-136c-435a-9029-b37773fd6088"
-      (reference "TP?") (unit 1) (value "TestPoint") (footprint "TestPoint:TestPoint_Pad_2.5x2.5mm")
+      (reference "TP1") (unit 1) (value "TestPoint") (footprint "TestPoint:TestPoint_Pad_2.5x2.5mm")
     )
   )
